File: ULN2803 RELAY BOARD.kicad_pcb (KiCad board)
At the start: 2 copper layers, 93 x 110 mm, 69 parts, among them J1 POWER, J10 NC CO NO, J2 INPUTS, J3 NC CO NO, J4 NC CO NO, J5 NC CO NO, J6 NC CO NO, J7 NC CO NO, J8 NC CO NO, J9 NC CO NO, K1 G5LE-1, K2 G5LE-1, K3 G5LE-1, K4 G5LE-1, K5 G5LE-1, K6 G5LE-1, K7 G5LE-1, K8 G5LE-1, SW1 SW_SPST, U1 ULN2803A

Commit message: Görseller eklendi
Parts:
- moved H1 2.00 mm to (97.0, 145.0)
- moved H2 2.00 mm to (178.0, 145.0)
- moved H3 2.00 mm to (97.0, 44.0)
- moved H4 2.00 mm to (178.0, 44.0)
Changed lines of the file:
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@@
 	(footprint "MountingHole:MountingHole_2.5mm_Pad_Via"
 		(layer "F.Cu")
-		(at 178 147 90)
+		(at 178 145 90)
 		(descr "Mounting Hole 2.5mm")
 		(tags "mounting hole 2.5mm")
@@
 	(footprint "MountingHole:MountingHole_2.5mm_Pad_Via"
 		(layer "F.Cu")
-		(at 178 46 90)
+		(at 178 44 90)
 		(descr "Mounting Hole 2.5mm")
 		(tags "mounting hole 2.5mm")
@@
 	(footprint "MountingHole:MountingHole_2.5mm_Pad_Via"
 		(layer "F.Cu")
-		(at 97 147 90)
+		(at 97 145 90)
 		(descr "Mounting Hole 2.5mm")
 		(tags "mounting hole 2.5mm")
@@
 	(footprint "MountingHole:MountingHole_2.5mm_Pad_Via"
 		(layer "F.Cu")
-		(at 97 46 90)
+		(at 97 44 90)
 		(descr "Mounting Hole 2.5mm")
 		(tags "mounting hole 2.5mm")
@@
 		(tags "Omron Relay SPDT")
 		(property "Reference" "K6"
-			(at 0 21 0)
+			(at 0 20.5 0)
 			(layer "F.SilkS")
 			(effects
@@
 	)
 	(gr_line
-		(start 96 41)
-		(end 179 41)
+		(start 96 39)
+		(end 179 39)
 		(stroke
 			(width 0.05)
@@
 	)
 	(gr_arc
-		(start 91 46)
-		(mid 92.464466 42.464466)
-		(end 96 41)
+		(start 91 44)
+		(mid 92.464466 40.464466)
+		(end 96 39)
 		(stroke
 			(width 0.05)
@@
 	)
 	(gr_line
-		(start 184 46)
-		(end 184 146)
+		(start 184 44)
+		(end 184 144)
 		(stroke
 			(width 0.05)
@@
 	)
 	(gr_line
-		(start 91 146)
-		(end 91 46)
+		(start 91 144)
+		(end 91 44)
 		(stroke
 			(width 0.05)
@@
 	)
 	(gr_arc
-		(start 179 41)
-		(mid 182.535534 42.464466)
-		(end 184 46)
+		(start 179 39)
+		(mid 182.535534 40.464466)
+		(end 184 44)
 		(stroke
 			(width 0.05)
@@
 	)
 	(gr_line
-		(start 179 151)
-		(end 96 151)
+		(start 179 149)
+		(end 96 149)
 		(stroke
 			(width 0.05)
@@
 	)
 	(gr_arc
-		(start 96 151)
-		(mid 92.464466 149.535534)
-		(end 91 146)
+		(start 96 149)
+		(mid 92.464466 147.535534)
+		(end 91 144)
 		(stroke
 			(width 0.05)
@@
 	)
 	(gr_arc
-		(start 184 146)
-		(mid 182.535534 149.535534)
-		(end 179 151)
+		(start 184 144)
+		(mid 182.535534 147.535534)
+		(end 179 149)
 		(stroke
 			(width 0.05)
@@
 		(polygon
 			(pts
-				(xy 101 42) (xy 175.5 42) (xy 175 149.5) (xy 100.5 149.5)
+				(xy 101 40) (xy 175.5 40) (xy 175 147.5) (xy 100.5 147.5)
 			)
 		)
@@
 		(polygon
 			(pts
-				(xy 94 150) (xy 181 150) (xy 181 43) (xy 94 43)
+				(xy 94 148) (xy 181 148) (xy 181 41) (xy 94 41)
 			)
 		)

Commit message: Baskı için güncellemeler yapıldı
Parts:
- D1: footprint LED_SMD:LED_0805_2012Metric -> LED_SMD:LED_1206_3216Metric
- D10, D12, D14, D16, D2, D4, D6, D8: footprint Diode_SMD:D_1206_3216Metric -> Diode_SMD:D_SMA
- R1, R18, R19, R20, R21, R22, R23, R24, R25: value 680 -> 680R
- SW1: footprint Button_Switch_SMD:SW_DIP_SPSTx01_Slide_6.7x4.1mm_W6.73mm_P2.54mm_LowProfile_JPin -> Button_Switch_THT:SW_DIP_SPSTx01_Slide_9.78x4.72mm_W7.62mm_P2.54mm
- moved SW1 4.03 mm to (164.2, 96.0)
- moved C2 1.60 mm to (151.6, 86.0)
- moved C3 1.60 mm to (155.0, 86.0)
- moved C1 1.31 mm to (159.0, 97.0)
- moved D5 1.28 mm to (129.4, 106.0)
- moved D2 1.12 mm to (104.0, 106.0)
- moved R1 1.09 mm to (159.0, 86.9)
- moved D3 1.00 mm to (110.9, 106.0)
- moved D4 1.00 mm to (122.4, 106.0)
- moved R18 0.93 mm to (115.9, 106.0)
- moved D9 0.86 mm to (165.1, 106.5)
- moved D7 0.78 mm to (147.1, 106.5)
- moved R19 0.78 mm to (134.4, 106.0)
- moved D13 0.70 mm to (128.4, 81.0)
- moved D10 0.60 mm to (117.0, 81.0)
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Routing:
- net /O1: track 41.3 -> 44.9 mm
- net GND: track 45.4 -> 42.5 mm
- net /O8: track 35.9 -> 33.2 mm, vias 1 -> 0
- net /O7: track 19.5 -> 17.2 mm, vias 1 -> 0
- net VCC: track 13.7 -> 11.7 mm
- net /O6: track 22.3 -> 24.1 mm
- net /O5: track 37.0 -> 38.1 mm, vias 0 -> 1
- net Net-(D5-A): track 3.59 -> 2.70 mm
- net /O3: track 55.3 -> 56.1 mm
- net Net-(D9-A): track 3.38 -> 2.68 mm
- net Net-(D13-A): track 3.29 -> 2.59 mm
- net Net-(D7-A): track 3.19 -> 2.50 mm
- net Net-(D1-A): track 2.00 -> 2.62 mm
- net Net-(D3-A): track 3.29 -> 2.70 mm
- net /O4: track 49.1 -> 49.7 mm
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